Commit message: Working moving robot example, readme

File: src/urdf_test/urdf/test_puzzlebot.urdf (robot description, URDF)
Before this commit: robot puzzlebot, 1 links, 0 joints
Links:
- added link l_wheel; visual mesh filename=package://urdf_test/meshes/MCR2_1000_1_1_Wheel_Coupler_2.stl
- added link r_wheel; visual mesh filename=package://urdf_test/meshes/MCR2_1000_1_1_Wheel_Coupler_2.stl
- link base_link: geometry visual mesh filename=package://urdf_test/meshes/MCR2_1000_13_Chassis.stl
Joints:
- added joint chassis_to_l_wheel: type continuous, parent base_link, child l_wheel, origin xyz=-0.085 -0.05 0, axis -1 0 0
- added joint chassis_to_r_wheel: type continuous, parent base_link, child r_wheel, origin xyz=0.085 -0.05 0, axis -1 0 0
